File: _autosave-kbic65.kicad_pcb (KiCad board)
At the start: 2 copper layers, 150 parts, among them U1 ProMicro

Commit message: Redrew schematic with all extra footprints
Parts:
- removed MX_BKSLSH2(ISO_Enter): MX-NoLED, MX_Only:MXOnly-ISO-ROTATED-ReversedStabilizers-NoLED
- removed MX_BkSp2(RegBkSp): MX-NoLED, MX_Only:MXOnly-2U-NoLED
- removed MX_CpsLck2(Stepped), MX_RAlt2, MX_RAlt3, MX_RWin2(RCtrl2): MX-NoLED, MX_Only:MXOnly-1.25U-NoLED
- removed MX_Enter2(ISO_Hash): MX-NoLED, MX_Only:MXOnly-1U-NoLED
- removed MX_LShift2(ANSI): MX-NoLED, MX_Only:MXOnly-2.25U-NoLED
- removed MX_Space2: MX-NoLED, MX_Only:MXOnly-6U-Centered-NoLED
