File: kbic65.sch (KiCad schematic (older format))
At the start: 141 parts, among them U1 ProMicro

Commit message: Redrew schematic with all extra footprints
Parts:
- added MX_BkSlash2_ISO_Enter: MX-NoLED, MX_Only:MXOnly-1.5U-NoLED, symbol MX_Alps_Hybrid:MX-NoLED
- added MX_BkSp3_2u, MX_RAlt2_1.25u_6u_space, MX_RAlt3_1.25u_6.25u_space, MX_RWin2_1.25u_RCtrl: MX-NoLED, MX_Only:MXOnly-1U-NoLED, symbol MX_Alps_Hybrid:MX-NoLED
- added MX_CpsLck2_Stepped: MX-NoLED, MX_Only:MXOnly-1.75U-NoLED, symbol MX_Alps_Hybrid:MX-NoLED
- added MX_Enter2_ISO_Hash: MX-NoLED, MX_Only:MXOnly-2.25U-NoLED, symbol MX_Alps_Hybrid:MX-NoLED
- added MX_LShift_ANSI: MX-NoLED, MX_Only:MXOnly-1.25U-NoLED, symbol MX_Alps_Hybrid:MX-NoLED
- added MX_Space2_6u: MX-NoLED, MX_Only:MXOnly-6.25U-NoLED, symbol MX_Alps_Hybrid:MX-NoLED
- MX_BkSlsh1: renamed from MX_BKSLSH1; footprint MX_Only:MXOnly-1U-NoLED -> MX_Only:MXOnly-1.5U-NoLED
- MX_CpsLck1, MX_RShift1: footprint MX_Only:MXOnly-1U-NoLED -> MX_Only:MXOnly-1.75U-NoLED
- MX_Enter1: footprint MX_Only:MXOnly-1U-NoLED -> MX_Only:MXOnly-2.25U-NoLED
- MX_LAlt1, MX_LCtrl1, MX_LWin1: footprint MX_Only:MXOnly-1U-NoLED -> MX_Only:MXOnly-1.25U-NoLED
- MX_LShift_ISO: renamed from MX_LShift1; footprint MX_Only:MXOnly-1U-NoLED -> MX_Only:MXOnly-1.25U-NoLED
- MX_Space1_6.25u: renamed from MX_Space1; footprint MX_Only:MXOnly-1U-NoLED -> MX_Only:MXOnly-6.25U-NoLED
- MX_Tab1: footprint MX_Only:MXOnly-1U-NoLED -> MX_Only:MXOnly-1.5U-NoLED
- renumbered MX_RAlt1 to MX_RAlt1_1u
Connections:
- net COL0: now also MX_CpsLck2_Stepped.1 (COL), MX_LShift_ANSI.1 (COL)
- net COL3: now also MX_Space2_6u.1 (COL)
- net COL4: no longer MX_RAlt1_1u.1 (COL)
- net COL5: now also MX_RWin2_1.25u_RCtrl.1 (COL)
- net COL6: now also MX_BkSlash2_ISO_Enter.1 (COL), MX_BkSp3_2u.1 (COL), MX_Enter2_ISO_Hash.1 (COL)
- net at D_BkSp1.2 (A), MX_BkSp1.2 (ROW): now also MX_BkSp3_2u.2 (ROW)
- net at D_BKSLSH1.2 (A), MX_BkSlsh1.2 (ROW): now also MX_BkSlash2_ISO_Enter.2 (ROW)
- net at D_CpsLck1.2 (A), MX_CpsLck1.2 (ROW): now also MX_CpsLck2_Stepped.2 (ROW)
- net at D_LShift1.2 (A), MX_LShift_ISO.2 (ROW): now also MX_LShift_ANSI.2 (ROW)
- net at D_Enter1.2 (A), MX_Enter1.2 (ROW): now also MX_Enter2_ISO_Hash.2 (ROW)
- net at D_Space1.2 (A), MX_Space1_6.25u.2 (ROW): now also MX_Space2_6u.2 (ROW)
- net at D_RAlt1.2 (A), MX_RAlt1_1u.2 (ROW): now also MX_RAlt2_1.25u_6u_space.2 (ROW), MX_RAlt3_1.25u_6.25u_space.2 (ROW)
- net at D_RWin1.2 (A), MX_RWin1.2 (ROW): now also MX_RWin2_1.25u_RCtrl.2 (ROW)
- new net: MX_RAlt1_1u.1 (COL), MX_RAlt2_1.25u_6u_space.1 (COL), MX_RAlt3_1.25u_6.25u_space.1 (COL)
Other:
- moved on the sheet: D_0, D_1, D_2, D_3, D_4, D_5, D_6, D_7, D_8, D_9, D_@1, D_A1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

Commit message: Changed layout to top windows and rearranging diodes
Parts:
- MX_BkSlash2_ISO_Enter1: renamed from MX_BkSlash2_ISO_Enter; footprint MX_Only:MXOnly-1.5U-NoLED -> MX_Only:MXOnly-ISO-ROTATED-ReversedStabilizers-NoLED
- MX_BkSp3_2u1: renamed from MX_BkSp3_2u; footprint MX_Only:MXOnly-1U-NoLED -> MX_Only:MXOnly-2U-NoLED
- MX_CpsLck2_Stepped1: renamed from MX_CpsLck2_Stepped; footprint MX_Only:MXOnly-1.75U-NoLED -> MX_Only:MXOnly-1.25U-NoLED
- MX_Enter2_ISO_Hash1: renamed from MX_Enter2_ISO_Hash; footprint MX_Only:MXOnly-2.25U-NoLED -> MX_Only:MXOnly-1U-NoLED
- MX_LShift_ANSI1: renamed from MX_LShift_ANSI; footprint MX_Only:MXOnly-1.25U-NoLED -> MX_Only:MXOnly-2.25U-NoLED
- MX_RAlt2_1.25u_6u_space1: renamed from MX_RAlt2_1.25u_6u_space; footprint MX_Only:MXOnly-1U-NoLED -> MX_Only:MXOnly-1.25U-NoLED
- MX_RAlt3_1.25u_6.25u_space1: renamed from MX_RAlt3_1.25u_6.25u_space; footprint MX_Only:MXOnly-1U-NoLED -> MX_Only:MXOnly-1.25U-NoLED
- MX_Space2_6u1: renamed from MX_Space2_6u; footprint MX_Only:MXOnly-6.25U-NoLED -> MX_Only:MXOnly-6U-Centered-NoLED
- renumbered MX_LShift_ISO to MX_LShift_ISO1, MX_RAlt1_1u to MX_RAlt1_1u1, MX_RWin2_1.25u_RCtrl to MX_RWin2_1.25u_RCtrl1, MX_Space1_6.25u to MX_Space1_6.25u1
Changed lines of the file:
@@
 	13450 8300 13550 8300
 $Comp
-L MX_Alps_Hybrid:MX-NoLED MX_LShift_ISO
+L MX_Alps_Hybrid:MX-NoLED MX_LShift_ISO1
 U 1 1 5FE8C66D
 P 12600 8150
-F 0 "MX_LShift_ISO" H 12633 8373 60  0000 C CNN
+F 0 "MX_LShift_ISO1" H 12633 8373 60  0000 C CNN
 F 1 "MX-NoLED" H 12633 8299 20  0000 C CNN
 F 2 "MX_Only:MXOnly-1.25U-NoLED" H 11975 8125 60  0001 C CNN
@@
 	14450 10200 14550 10200
 $Comp
-L MX_Alps_Hybrid:MX-NoLED MX_Space1_6.25u
+L MX_Alps_Hybrid:MX-NoLED MX_Space1_6.25u1
 U 1 1 5FEAB46F
 P 18600 10050
-F 0 "MX_Space1_6.25u" H 18633 10273 60  0000 C CNN
+F 0 "MX_Space1_6.25u1" H 18633 10273 60  0000 C CNN
 F 1 "MX-NoLED" H 18633 10199 20  0000 C CNN
 F 2 "MX_Only:MXOnly-6.25U-NoLED" H 17975 10025 60  0001 C CNN
@@
 	18450 10200 18550 10200
 $Comp
-L MX_Alps_Hybrid:MX-NoLED MX_RAlt1_1u
+L MX_Alps_Hybrid:MX-NoLED MX_RAlt1_1u1
 U 1 1 5FEAB47C
 P 22600 10050
-F 0 "MX_RAlt1_1u" H 22633 10273 60  0000 C CNN
+F 0 "MX_RAlt1_1u1" H 22633 10273 60  0000 C CNN
 F 1 "MX-NoLED" H 22633 10199 20  0000 C CNN
 F 2 "MX_Only:MXOnly-1U-NoLED" H 21975 10025 60  0001 C CNN
@@
 $EndComp
 $Comp
-L MX_Alps_Hybrid:MX-NoLED MX_LShift_ANSI
+L MX_Alps_Hybrid:MX-NoLED MX_LShift_ANSI1
 U 1 1 5FDB85B5
 P 11750 8150
-F 0 "MX_LShift_ANSI" H 11783 8373 60  0000 C CNN
+F 0 "MX_LShift_ANSI1" H 11783 8373 60  0000 C CNN
 F 1 "MX-NoLED" H 11783 8299 20  0000 C CNN
-F 2 "MX_Only:MXOnly-1.25U-NoLED" H 11125 8125 60  0001 C CNN
+F 2 "MX_Only:MXOnly-2.25U-NoLED" H 11125 8125 60  0001 C CNN
 F 3 "" H 11125 8125 60  0001 C CNN
 	1    11750 8150
@@
 Connection ~ 12750 8100
 $Comp
-L MX_Alps_Hybrid:MX-NoLED MX_CpsLck2_Stepped
+L MX_Alps_Hybrid:MX-NoLED MX_CpsLck2_Stepped1
 U 1 1 5FDE4E7F
 P 11850 6700
-F 0 "MX_CpsLck2_Stepped" H 11883 6923 60  0000 C CNN
+F 0 "MX_CpsLck2_Stepped1" H 11883 6923 60  0000 C CNN
 F 1 "MX-NoLED" H 11883 6849 20  0000 C CNN
-F 2 "MX_Only:MXOnly-1.75U-NoLED" H 11225 6675 60  0001 C CNN
+F 2 "MX_Only:MXOnly-1.25U-NoLED" H 11225 6675 60  0001 C CNN
 F 3 "" H 11225 6675 60  0001 C CNN
 	1    11850 6700
@@
 $EndComp
 $Comp
-L MX_Alps_Hybrid:MX-NoLED MX_Space2_6u
+L MX_Alps_Hybrid:MX-NoLED MX_Space2_6u1
 U 1 1 5FE01F7D
 P 18600 11100
-F 0 "MX_Space2_6u" H 18633 11323 60  0000 C CNN
+F 0 "MX_Space2_6u1" H 18633 11323 60  0000 C CNN
 F 1 "MX-NoLED" H 18633 11249 20  0000 C CNN
-F 2 "MX_Only:MXOnly-6.25U-NoLED" H 17975 11075 60  0001 C CNN
+F 2 "MX_Only:MXOnly-6U-Centered-NoLED" H 17975 11075 60  0001 C CNN
 F 3 "" H 17975 11075 60  0001 C CNN
 	1    18600 11100
@@
 Connection ~ 18750 10000
 $Comp
-L MX_Alps_Hybrid:MX-NoLED MX_RAlt2_1.25u_6u_space
+L MX_Alps_Hybrid:MX-NoLED MX_RAlt2_1.25u_6u_space1
 U 1 1 5FE36BCB
 P 22600 10900
-F 0 "MX_RAlt2_1.25u_6u_space" H 22633 11123 60  0000 C CNN
+F 0 "MX_RAlt2_1.25u_6u_space1" H 22633 11123 60  0000 C CNN
 F 1 "MX-NoLED" H 22633 11049 20  0000 C CNN
-F 2 "MX_Only:MXOnly-1U-NoLED" H 21975 10875 60  0001 C CNN
+F 2 "MX_Only:MXOnly-1.25U-NoLED" H 21975 10875 60  0001 C CNN
 F 3 "" H 21975 10875 60  0001 C CNN
 	1    22600 10900
@@
 $EndComp
 $Comp
-L MX_Alps_Hybrid:MX-NoLED MX_RAlt3_1.25u_6.25u_space
+L MX_Alps_Hybrid:MX-NoLED MX_RAlt3_1.25u_6.25u_space1
 U 1 1 5FE370FA
 P 22600 11550
-F 0 "MX_RAlt3_1.25u_6.25u_space" H 22633 11773 60  0000 C CNN
+F 0 "MX_RAlt3_1.25u_6.25u_space1" H 22633 11773 60  0000 C CNN
 F 1 "MX-NoLED" H 22633 11699 20  0000 C CNN
-F 2 "MX_Only:MXOnly-1U-NoLED" H 21975 11525 60  0001 C CNN
+F 2 "MX_Only:MXOnly-1.25U-NoLED" H 21975 11525 60  0001 C CNN
 F 3 "" H 21975 11525 60  0001 C CNN
 	1    22600 11550
@@
 	22750 10850 22750 11500
 $Comp
-L MX_Alps_Hybrid:MX-NoLED MX_RWin2_1.25u_RCtrl
+L MX_Alps_Hybrid:MX-NoLED MX_RWin2_1.25u_RCtrl1
 U 1 1 5FE74F69
 P 23600 10950
-F 0 "MX_RWin2_1.25u_RCtrl" H 23633 11173 60  0000 C CNN
+F 0 "MX_RWin2_1.25u_RCtrl1" H 23633 11173 60  0000 C CNN
 F 1 "MX-NoLED" H 23633 11099 20  0000 C CNN
 F 2 "MX_Only:MXOnly-1U-NoLED" H 22975 10925 60  0001 C CNN
@@
 	23750 10000 23750 10900
 $Comp
-L MX_Alps_Hybrid:MX-NoLED MX_Enter2_ISO_Hash
+L MX_Alps_Hybrid:MX-NoLED MX_Enter2_ISO_Hash1
 U 1 1 5FE93AC3
 P 25300 6700
-F 0 "MX_Enter2_ISO_Hash" H 25333 6923 60  0000 C CNN
+F 0 "MX_Enter2_ISO_Hash1" H 25333 6923 60  0000 C CNN
 F 1 "MX-NoLED" H 25333 6849 20  0000 C CNN
-F 2 "MX_Only:MXOnly-2.25U-NoLED" H 24675 6675 60  0001 C CNN
+F 2 "MX_Only:MXOnly-1U-NoLED" H 24675 6675 60  0001 C CNN
 F 3 "" H 24675 6675 60  0001 C CNN
 	1    25300 6700
@@
 Connection ~ 24550 6850
 $Comp
-L MX_Alps_Hybrid:MX-NoLED MX_BkSlash2_ISO_Enter
+L MX_Alps_Hybrid:MX-NoLED MX_BkSlash2_ISO_Enter1
 U 1 1 5FEB466D
 P 26650 5300
-F 0 "MX_BkSlash2_ISO_Enter" H 26683 5523 60  0000 C CNN
+F 0 "MX_BkSlash2_ISO_Enter1" H 26683 5523 60  0000 C CNN
 F 1 "MX-NoLED" H 26683 5449 20  0000 C CNN
-F 2 "MX_Only:MXOnly-1.5U-NoLED" H 26025 5275 60  0001 C CNN
+F 2 "MX_Only:MXOnly-ISO-ROTATED-ReversedStabilizers-NoLED" H 26025 5275 60  0001 C CNN
 F 3 "" H 26025 5275 60  0001 C CNN
 	1    26650 5300
@@
 $EndComp
 $Comp
-L MX_Alps_Hybrid:MX-NoLED MX_BkSp3_2u
+L MX_Alps_Hybrid:MX-NoLED MX_BkSp3_2u1
 U 1 1 5FEB7A51
 P 25600 3500
-F 0 "MX_BkSp3_2u" H 25633 3723 60  0000 C CNN
+F 0 "MX_BkSp3_2u1" H 25633 3723 60  0000 C CNN
 F 1 "MX-NoLED" H 25633 3649 20  0000 C CNN
-F 2 "MX_Only:MXOnly-1U-NoLED" H 24975 3475 60  0001 C CNN
+F 2 "MX_Only:MXOnly-2U-NoLED" H 24975 3475 60  0001 C CNN
 F 3 "" H 24975 3475 60  0001 C CNN
 	1    25600 3500
