File: kbic65.kicad_pcb (KiCad board)
At the start: 2 copper layers, 150 parts, among them U1 ProMicro

Commit message: Reverted back to single line of diodes
Parts:
- moved D_Tilde1 23.2 mm to (359.6, 52.4)
- moved D_Del1 22.7 mm to (356.1, 52.4)
- moved D_PgUp1 22.3 mm to (352.6, 52.4)
- moved D_PgDn1 21.8 mm to (349.1, 52.4)
- moved D_Right1 21.3 mm to (345.7, 52.4)
- moved D_Down1 20.8 mm to (342.2, 52.4)
- moved D_Left1 20.3 mm to (338.7, 52.4)
- moved D_BkSp1 20.1 mm to (331.8, 52.4)
- moved D_BkSp2 19.8 mm to (335.3, 52.4)
- moved D_BKSLSH1 19.6 mm to (328.3, 52.4)
- moved D_RBKT1 19.2 mm to (324.8, 52.4)
- moved D_Enter1 18.7 mm to (321.4, 52.4)
- moved D_Up1 18.2 mm to (317.9, 52.4)
- moved D_RShift1 17.8 mm to (314.4, 52.4)
- moved D_RCtrl1 17.3 mm to (310.9, 52.4)
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
Commit message: Changed outline to inkscape generated and aligned it
Parts:
- moved MX_9 33.9 mm to (227.0, 79.4)
- moved MX_@1 33.9 mm to (279.4, 117.5)
- moved MX_BkSp1 33.9 mm to (303.2, 79.4)
- moved MX_BkSp2 33.9 mm to (322.3, 79.4)
- moved MX_Del1 33.9 mm to (350.8, 98.4)
- moved MX_Dot1 33.9 mm to (250.8, 136.5)
- moved MX_Down1 33.9 mm to (327.0, 160.3)
- moved MX_Enter1 33.9 mm to (310.4, 117.5)
- moved MX_Enter2_ISO_Hash1 33.9 mm to (298.4, 117.5)
- moved MX_LBKT1 33.9 mm to (274.6, 98.4)
- moved MX_PgDn1 33.9 mm to (350.8, 136.5)
- moved MX_PgUp1 33.9 mm to (350.8, 117.5)
- moved MX_Right1 33.9 mm to (346.1, 160.3)
- moved MX_Tilde1 33.9 mm to (350.8, 79.4)
- moved MX_Up1 33.9 mm to (327.0, 141.3)
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
Commit message: Finally started wiring
Routing:
- net Net-(D_Left1-Pad2): track 0.00 -> 143.4 mm
- net Net-(D_Down1-Pad2): track 0.00 -> 126.2 mm
- net Net-(D_Right1-Pad2): track 0.00 -> 119.8 mm
- net Net-(D_PgDn1-Pad2): track 0.00 -> 95.4 mm
- net Net-(D_PgUp1-Pad2): track 0.00 -> 73.8 mm
- net Net-(D_Del1-Pad2): track 0.00 -> 52.2 mm
- net Net-(D_Tilde1-Pad2): track 0.00 -> 31.6 mm
- net Net-(D_BkSp2-Pad2): track 0.00 -> 25.9 mm
- net Net-(D_BkSp1-Pad2): track 0.00 -> 19.1 mm
- net Net-(D_BKSLSH1-Pad2): track 0.00 -> 14.4 mm
Changed lines of the file:
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@@
     (thickness 1.6)
     (drawings 928)
-    (tracks 0)
+    (tracks 45)
     (zones 0)
     (modules 150)
@@
     (pad_to_mask_clearance 0)
     (aux_axis_origin 0 0)
-    (visible_elements 7FFDF7FF)
+    (visible_elements 7FFDFFFF)
     (pcbplotparams
       (layerselection 0x010fc_ffffffff)
@@
   (gr_line (start 62.562499 72.374992) (end 62.562499 86.375408) (layer Dwgs.User) (width 0.2))
   (gr_line (start 48.562083 72.374992) (end 62.562499 72.374992) (layer Dwgs.User) (width 0.2))
+  (segment (start 318.391974 95.885) (end 313.945151 95.885) (width 0.25) (layer B.Cu) (net 18))
+  (segment (start 321.296251 98.789277) (end 318.391974 95.885) (width 0.25) (layer B.Cu) (net 18))
+  (segment (start 321.296251 103.015001) (end 321.296251 98.789277) (width 0.25) (layer B.Cu) (net 18))
+  (segment (start 322.42125 104.14) (end 321.296251 103.015001) (width 0.25) (layer B.Cu) (net 18))
+  (segment (start 298.277501 58.422233) (end 298.438484 58.26125) (width 0.25) (layer B.Cu) (net 20))
+  (segment (start 298.277501 75.710001) (end 298.277501 58.422233) (width 0.25) (layer B.Cu) (net 20))
+  (segment (start 299.4025 76.835) (end 298.277501 75.710001) (width 0.25) (layer B.Cu) (net 20))
+  (segment (start 318.4525 76.835) (end 318.4525 73.9775) (width 0.25) (layer B.Cu) (net 21))
+  (segment (start 302.73625 58.26125) (end 301.912578 58.26125) (width 0.25) (layer B.Cu) (net 21))
+  (segment (start 318.4525 73.9775) (end 302.73625 58.26125) (width 0.25) (layer B.Cu) (net 21))
+  (segment (start 347.0275 95.885) (end 343.69375 92.55125) (width 0.25) (layer B.Cu) (net 28))
+  (segment (start 343.69375 92.55125) (end 343.69375 71.4375) (width 0.25) (layer B.Cu) (net 28))
+  (segment (start 343.69375 71.4375) (end 332.58125 60.325) (width 0.25) (layer B.Cu) (net 28))
+  (segment (start 324.820892 60.325) (end 322.757142 58.26125) (width 0.25) (layer B.Cu) (net 28))
+  (segment (start 332.58125 60.325) (end 324.820892 60.325) (width 0.25) (layer B.Cu) (net 28))
+  (segment (start 323.215 157.7975) (end 337.34375 143.66875) (width 0.25) (layer B.Cu) (net 31))
+  (segment (start 337.34375 143.66875) (end 337.34375 71.4375) (width 0.25) (layer B.Cu) (net 31))
+  (segment (start 337.34375 71.4375) (end 332.58125 66.675) (width 0.25) (layer B.Cu) (net 31))
+  (segment (start 332.58125 66.675) (end 317.5 66.675) (width 0.25) (layer B.Cu) (net 31))
+  (segment (start 309.08625 58.26125) (end 308.860766 58.26125) (width 0.25) (layer B.Cu) (net 31))
+  (segment (start 317.5 66.675) (end 309.08625 58.26125) (width 0.25) (layer B.Cu) (net 31))
+  (segment (start 331.7875 68.2625) (end 315.387922 68.2625) (width 0.25) (layer B.Cu) (net 50))
+  (segment (start 334.9625 71.4375) (end 331.7875 68.2625) (width 0.25) (layer B.Cu) (net 50))
+  (segment (start 334.9625 142.875) (end 334.9625 71.4375) (width 0.25) (layer B.Cu) (net 50))
+  (segment (start 315.387922 68.2625) (end 305.386672 58.26125) (width 0.25) (layer B.Cu) (net 50))
+  (segment (start 320.04 157.7975) (end 334.9625 142.875) (width 0.25) (layer B.Cu) (net 50))
+  (segment (start 304.165 157.7975) (end 320.04 157.7975) (width 0.25) (layer B.Cu) (net 50))
+  (segment (start 321.047704 63.5) (end 315.808954 58.26125) (width 0.25) (layer B.Cu) (net 57))
+  (segment (start 332.58125 63.5) (end 321.047704 63.5) (width 0.25) (layer B.Cu) (net 57))
+  (segment (start 340.51875 71.4375) (end 332.58125 63.5) (width 0.25) (layer B.Cu) (net 57))
+  (segment (start 340.51875 127.47625) (end 340.51875 71.4375) (width 0.25) (layer B.Cu) (net 57))
+  (segment (start 347.0275 133.985) (end 340.51875 127.47625) (width 0.25) (layer B.Cu) (net 57))
+  (segment (start 347.0275 114.935) (end 342.10625 110.01375) (width 0.25) (layer B.Cu) (net 58))
+  (segment (start 342.10625 110.01375) (end 342.10625 71.4375) (width 0.25) (layer B.Cu) (net 58))
+  (segment (start 342.10625 71.4375) (end 332.58125 61.9125) (width 0.25) (layer B.Cu) (net 58))
+  (segment (start 322.934298 61.9125) (end 319.283048 58.26125) (width 0.25) (layer B.Cu) (net 58))
+  (segment (start 332.58125 61.9125) (end 322.934298 61.9125) (width 0.25) (layer B.Cu) (net 58))
+  (segment (start 332.58125 65.0875) (end 319.16111 65.0875) (width 0.25) (layer B.Cu) (net 64))
+  (segment (start 338.93125 71.4375) (end 332.58125 65.0875) (width 0.25) (layer B.Cu) (net 64))
+  (segment (start 338.93125 154.46375) (end 338.93125 71.4375) (width 0.25) (layer B.Cu) (net 64))
+  (segment (start 319.16111 65.0875) (end 312.33486 58.26125) (width 0.25) (layer B.Cu) (net 64))
+  (segment (start 342.265 157.7975) (end 338.93125 154.46375) (width 0.25) (layer B.Cu) (net 64))
+  (segment (start 347.0275 76.835) (end 347.0275 71.59625) (width 0.25) (layer B.Cu) (net 72))
+  (segment (start 333.6925 58.26125) (end 326.23125 58.26125) (width 0.25) (layer B.Cu) (net 72))
+  (segment (start 347.0275 71.59625) (end 333.6925 58.26125) (width 0.25) (layer B.Cu) (net 72))
 )
