File: kicad/kbic65.kicad_pcb (KiCad board)
At the start: 2 copper layers, 313.3 x 123.8 mm, 154 parts, among them U1 ProMicro

Commit message: Updated board design and rewired, starting silkscreens
Parts:
- removed D_0, D_1, D_2, D_3, D_4, D_5, D_6, D_7, D_8, D_9, D_@1, D_A1, D_B1, D_BKSLSH1, D_BkSp1, D_BkSp2, D_C1, D_Comma1, D_CpsLck1, D_D1, D_Del1, D_Dot1, D_Down1, D_E1, D_Enter1, D_Equal1, D_Esc1, D_F1, D_FwdSlsh1, D_G1, D_H1, D_Hyphen1, D_I1, D_ISO_BKSLSH1, D_J1, D_K1, D_L1, D_LAlt1, D_LBKT1, D_LCtrl1, D_LShift1, D_LWin1, D_Left1, D_M1, D_N1, D_O1, D_P1, D_PgDn1, D_PgUp1, D_Q1, D_R1, D_RAlt1, D_RBKT1, D_RCtrl1, D_RShift1, D_RWin1, D_Right1, D_S1, D_SemiCol1, D_Space1, D_T1, D_Tab1, D_Tilde1, D_U1, D_Up1, D_V1, D_W1, D_X1, D_Y1, D_Z1: SOD_123, Diode_THT:D_DO-35_SOD27_P5.08mm_Vertical_AnodeUp
- removed MX_BkSp2, MX_Esc1, MX_G1: MX-NoLED, MX_Only:MXOnly-1U-NoLED
- removed MX_BkSp3_2u1: MX-NoLED, MX_Only:MXOnly-2U-NoLED
- removed the REF** at (355.6, 67.5)
- removed the REF** at (254.0, 67.5)
- removed the REF** at (152.4, 67.5)
- removed the REF** at (50.8, 67.5)
- added #: SOD_123, Diode_THT:D_DO-35_SOD27_P5.08mm_Vertical_AnodeUp, F.Cu at (281.1, 47.6)
- added ': SOD_123, Diode_THT:D_DO-35_SOD27_P5.08mm_Vertical_AnodeUp, F.Cu at (261.1, 47.6)
- added ,: SOD_123, Diode_THT:D_DO-35_SOD27_P5.08mm_Vertical_AnodeUp, F.Cu at (224.5, 47.6)
- added -: SOD_123, Diode_THT:D_DO-35_SOD27_P5.08mm_Vertical_AnodeUp, F.Cu at (241.1, 47.6)
- added .: SOD_123, Diode_THT:D_DO-35_SOD27_P5.08mm_Vertical_AnodeUp, F.Cu at (251.1, 47.6)
- added /: SOD_123, Diode_THT:D_DO-35_SOD27_P5.08mm_Vertical_AnodeUp, F.Cu at (257.8, 47.6)
- added 0: SOD_123, Diode_THT:D_DO-35_SOD27_P5.08mm_Vertical_AnodeUp, F.Cu at (237.8, 47.6)
- added 1: SOD_123, Diode_THT:D_DO-35_SOD27_P5.08mm_Vertical_AnodeUp, F.Cu at (87.8, 47.6)
- added 2: SOD_123, Diode_THT:D_DO-35_SOD27_P5.08mm_Vertical_AnodeUp, F.Cu at (131.1, 47.6)
- added 3: SOD_123, Diode_THT:D_DO-35_SOD27_P5.08mm_Vertical_AnodeUp, F.Cu at (134.4, 47.6)
- added 4: SOD_123, Diode_THT:D_DO-35_SOD27_P5.08mm_Vertical_AnodeUp, F.Cu at (161.1, 47.6)
- added 5: SOD_123, Diode_THT:D_DO-35_SOD27_P5.08mm_Vertical_AnodeUp, F.Cu at (164.4, 47.6)
- added 6: SOD_123, Diode_THT:D_DO-35_SOD27_P5.08mm_Vertical_AnodeUp, F.Cu at (177.8, 47.6)
- added 7: SOD_123, Diode_THT:D_DO-35_SOD27_P5.08mm_Vertical_AnodeUp, F.Cu at (181.1, 47.6)
- added 8: SOD_123, Diode_THT:D_DO-35_SOD27_P5.08mm_Vertical_AnodeUp, F.Cu at (207.8, 47.6)
- added 9: SOD_123, Diode_THT:D_DO-35_SOD27_P5.08mm_Vertical_AnodeUp, F.Cu at (211.1, 47.6)
- added ;: SOD_123, Diode_THT:D_DO-35_SOD27_P5.08mm_Vertical_AnodeUp, F.Cu at (247.8, 47.6)
- added =: SOD_123, Diode_THT:D_DO-35_SOD27_P5.08mm_Vertical_AnodeUp, F.Cu at (267.8, 47.6)
- added A: SOD_123, Diode_THT:D_DO-35_SOD27_P5.08mm_Vertical_AnodeUp, F.Cu at (94.4, 47.6)
- added B: SOD_123, Diode_THT:D_DO-35_SOD27_P5.08mm_Vertical_AnodeUp, F.Cu at (191.1, 47.6)
- added Backpace 2: MX-NoLED, MX_Only:MXOnly-1U-NoLED, F.Cu at (322.3, 79.4)
- added BkSp: SOD_123, Diode_THT:D_DO-35_SOD27_P5.08mm_Vertical_AnodeUp, F.Cu at (291.1, 47.6)
- added BkSp 3: MX-NoLED, MX_Only:MXOnly-2U-NoLED, F.Cu at (312.7, 79.4)
- added BkSp2: SOD_123, Diode_THT:D_DO-35_SOD27_P5.08mm_Vertical_AnodeUp, F.Cu at (294.5, 47.6)
- added C: SOD_123, Diode_THT:D_DO-35_SOD27_P5.08mm_Vertical_AnodeUp, F.Cu at (151.1, 47.6)
- added CpsLck: SOD_123, Diode_THT:D_DO-35_SOD27_P5.08mm_Vertical_AnodeUp, F.Cu at (104.4, 47.6)
- added D: SOD_123, Diode_THT:D_DO-35_SOD27_P5.08mm_Vertical_AnodeUp, F.Cu at (141.1, 47.6)
- added Del: SOD_123, Diode_THT:D_DO-35_SOD27_P5.08mm_Vertical_AnodeUp, F.Cu at (314.5, 47.6)
- added Down: SOD_123, Diode_THT:D_DO-35_SOD27_P5.08mm_Vertical_AnodeUp, F.Cu at (301.1, 47.6)
- added E: SOD_123, Diode_THT:D_DO-35_SOD27_P5.08mm_Vertical_AnodeUp, F.Cu at (137.8, 47.6)
- added Esc: MX-NoLED, MX_Only:MXOnly-1U-NoLED, F.Cu at (55.6, 79.4)
- added Esc: SOD_123, Diode_THT:D_DO-35_SOD27_P5.08mm_Vertical_AnodeUp, F.Cu at (111.1, 47.6)
- added F: SOD_123, Diode_THT:D_DO-35_SOD27_P5.08mm_Vertical_AnodeUp, F.Cu at (154.4, 47.6)
- added G: MX-NoLED, MX_Only:MXOnly-1U-NoLED, F.Cu at (165.1, 117.5)
- added G: SOD_123, Diode_THT:D_DO-35_SOD27_P5.08mm_Vertical_AnodeUp, F.Cu at (171.1, 47.6)
- added H: SOD_123, Diode_THT:D_DO-35_SOD27_P5.08mm_Vertical_AnodeUp, F.Cu at (187.8, 47.6)
- added I: SOD_123, Diode_THT:D_DO-35_SOD27_P5.08mm_Vertical_AnodeUp, F.Cu at (214.5, 47.6)
- added J: SOD_123, Diode_THT:D_DO-35_SOD27_P5.08mm_Vertical_AnodeUp, F.Cu at (201.1, 47.6)
- added K: SOD_123, Diode_THT:D_DO-35_SOD27_P5.08mm_Vertical_AnodeUp, F.Cu at (217.8, 47.6)
- added L: SOD_123, Diode_THT:D_DO-35_SOD27_P5.08mm_Vertical_AnodeUp, F.Cu at (231.1, 47.6)
- added LAlt: SOD_123, Diode_THT:D_DO-35_SOD27_P5.08mm_Vertical_AnodeUp, F.Cu at (147.8, 47.6)
- added LCtrl: SOD_123, Diode_THT:D_DO-35_SOD27_P5.08mm_Vertical_AnodeUp, F.Cu at (114.4, 47.6)
- added LShift: SOD_123, Diode_THT:D_DO-35_SOD27_P5.08mm_Vertical_AnodeUp, F.Cu at (101.1, 47.6)
- added LWin: SOD_123, Diode_THT:D_DO-35_SOD27_P5.08mm_Vertical_AnodeUp, F.Cu at (117.8, 47.6)
- added Left: SOD_123, Diode_THT:D_DO-35_SOD27_P5.08mm_Vertical_AnodeUp, F.Cu at (297.8, 47.6)
- added M: SOD_123, Diode_THT:D_DO-35_SOD27_P5.08mm_Vertical_AnodeUp, F.Cu at (221.1, 47.6)
- added N: SOD_123, Diode_THT:D_DO-35_SOD27_P5.08mm_Vertical_AnodeUp, F.Cu at (197.8, 47.6)
- added O: SOD_123, Diode_THT:D_DO-35_SOD27_P5.08mm_Vertical_AnodeUp, F.Cu at (234.5, 47.6)
- added P: SOD_123, Diode_THT:D_DO-35_SOD27_P5.08mm_Vertical_AnodeUp, F.Cu at (244.5, 47.6)
- added PgDn: SOD_123, Diode_THT:D_DO-35_SOD27_P5.08mm_Vertical_AnodeUp, F.Cu at (307.8, 47.6)
- added PgUp: SOD_123, Diode_THT:D_DO-35_SOD27_P5.08mm_Vertical_AnodeUp, F.Cu at (311.2, 47.6)
- added Q: SOD_123, Diode_THT:D_DO-35_SOD27_P5.08mm_Vertical_AnodeUp, F.Cu at (91.1, 47.6)
- added R: SOD_123, Diode_THT:D_DO-35_SOD27_P5.08mm_Vertical_AnodeUp, F.Cu at (157.8, 47.6)
- added RAlt: SOD_123, Diode_THT:D_DO-35_SOD27_P5.08mm_Vertical_AnodeUp, F.Cu at (227.8, 47.6)
- added RCtrl: SOD_123, Diode_THT:D_DO-35_SOD27_P5.08mm_Vertical_AnodeUp, F.Cu at (271.1, 47.6)
- added REF**: MountingHole_5mm_Custom, KBIC-Parts:MountingHole_5mm_KB, F.Cu at (356.4, 67.5)
- added REF**: MountingHole_5mm_Custom, KBIC-Parts:MountingHole_5mm_KB, F.Cu at (254.8, 67.5)
- added REF**: MountingHole_5mm_Custom, KBIC-Parts:MountingHole_5mm_KB, F.Cu at (151.6, 67.5)
- added REF**: MountingHole_5mm_Custom, KBIC-Parts:MountingHole_5mm_KB, F.Cu at (50.0, 67.5)
- added RShift: SOD_123, Diode_THT:D_DO-35_SOD27_P5.08mm_Vertical_AnodeUp, F.Cu at (274.5, 47.6)
- added RWin: SOD_123, Diode_THT:D_DO-35_SOD27_P5.08mm_Vertical_AnodeUp, F.Cu at (254.5, 47.6)
- added Right: SOD_123, Diode_THT:D_DO-35_SOD27_P5.08mm_Vertical_AnodeUp, F.Cu at (304.5, 47.6)
- added S: SOD_123, Diode_THT:D_DO-35_SOD27_P5.08mm_Vertical_AnodeUp, F.Cu at (124.4, 47.6)
- added Space: SOD_123, Diode_THT:D_DO-35_SOD27_P5.08mm_Vertical_AnodeUp, F.Cu at (194.4, 47.6)
- added T: SOD_123, Diode_THT:D_DO-35_SOD27_P5.08mm_Vertical_AnodeUp, F.Cu at (174.4, 47.6)
- added Tab: SOD_123, Diode_THT:D_DO-35_SOD27_P5.08mm_Vertical_AnodeUp, F.Cu at (107.8, 47.6)
- added U: SOD_123, Diode_THT:D_DO-35_SOD27_P5.08mm_Vertical_AnodeUp, F.Cu at (204.5, 47.6)
- added Up: SOD_123, Diode_THT:D_DO-35_SOD27_P5.08mm_Vertical_AnodeUp, F.Cu at (277.8, 47.6)
- added V: SOD_123, Diode_THT:D_DO-35_SOD27_P5.08mm_Vertical_AnodeUp, F.Cu at (167.8, 47.6)
- added W: SOD_123, Diode_THT:D_DO-35_SOD27_P5.08mm_Vertical_AnodeUp, F.Cu at (127.8, 47.6)
- added X: SOD_123, Diode_THT:D_DO-35_SOD27_P5.08mm_Vertical_AnodeUp, F.Cu at (144.4, 47.6)
- added Y: SOD_123, Diode_THT:D_DO-35_SOD27_P5.08mm_Vertical_AnodeUp, F.Cu at (184.4, 47.6)
- added Z: SOD_123, Diode_THT:D_DO-35_SOD27_P5.08mm_Vertical_AnodeUp, F.Cu at (121.1, 47.6)
- added [: SOD_123, Diode_THT:D_DO-35_SOD27_P5.08mm_Vertical_AnodeUp, F.Cu at (264.5, 47.6)
- added \: SOD_123, Diode_THT:D_DO-35_SOD27_P5.08mm_Vertical_AnodeUp, F.Cu at (97.8, 47.6)
- added \: SOD_123, Diode_THT:D_DO-35_SOD27_P5.08mm_Vertical_AnodeUp, F.Cu at (287.8, 47.6)
- added ]: SOD_123, Diode_THT:D_DO-35_SOD27_P5.08mm_Vertical_AnodeUp, F.Cu at (284.5, 47.6)
- added ¬: SOD_123, Diode_THT:D_DO-35_SOD27_P5.08mm_Vertical_AnodeUp, F.Cu at (317.8, 47.6)
- Caps Lock: renamed from MX_CpsLck1
- Enter ANSI: renamed from MX_Enter1
- L Alt: renamed from MX_LAlt1
- L Ctrl: renamed from MX_LCtrl1
- L Shift: renamed from MX_LShift_ISO1
- L Win: renamed from MX_LWin1
- Page Down: renamed from MX_PgDn1
- Page Up: renamed from MX_PgUp1
- R Alt: renamed from MX_RAlt3_1.25u_6.25u_space1
- R Ctrl: renamed from MX_RCtrl1
- R Win: renamed from MX_RWin1
- \ ANSI: renamed from MX_BkSlsh1
- moved U1 5.78 mm to (65.9, 50.0)
- renumbered MX_Enter2_ISO_Hash1 to #, MX_@1 to ', MX_Comma1 to ,, MX_Hyphen1 to -, MX_Dot1 to ., MX_FwdSlsh1 to /, MX_0 to 0, MX_1 to 1, MX_2 to 2, MX_3 to 3, MX_4 to 4, MX_5 to 5, MX_6 to 6, MX_7 to 7, MX_8 to 8, MX_9 to 9, MX_SemiCol1 to ;, MX_Equal1 to =, MX_A1 to A, MX_B1 to B, MX_BkSp1 to Backspace, MX_C1 to C, MX_D1 to D, MX_Del1 to Delete, MX_Down1 to Down, MX_E1 to E, MX_BkSlash2_ISO_Enter1 to Enter, MX_F1 to F, MX_H1 to H, MX_I1 to I, MX_J1 to J, MX_K1 to K, MX_L1 to L, MX_Left1 to Left, MX_M1 to M, MX_N1 to N, MX_O1 to O, MX_P1 to P, MX_Q1 to Q, MX_R1 to R, MX_RShift1 to RShift, MX_Right1 to Right, MX_S1 to S, MX_Space1_6.25u1 to Space, MX_T1 to T, MX_Tab1 to Tab, MX_U1 to U, MX_Up1 to Up, MX_V1 to V, MX_W1 to W, MX_X1 to X, MX_Y1 to Y, MX_Z1 to Z, MX_LBKT1 to [, MX_ISO_BKSLSH1 to \, MX_RBKT1 to ], MX_Tilde1 to ¬
Routing:
- net Net-(D_5-Pad2): track 31.4 -> 45.7 mm
- net Net-(D_Equal1-Pad2): track 23.4 -> 35.2 mm
- net Net-(D_6-Pad2): track 39.8 -> 29.0 mm
- net Net-(D_BkSp1-Pad2): track 29.7 -> 40.3 mm
- net Net-(D_LBKT1-Pad2): track 42.5 -> 53.1 mm
- net Net-(D_BKSLSH1-Pad2): track 83.5 -> 93.8 mm
- net Net-(D_Comma1-Pad2): track 85.8 -> 95.8 mm
- net Net-(D_M1-Pad2): track 104.3 -> 114.2 mm
- net Net-(D_K1-Pad2): track 82.2 -> 92.0 mm
- net Net-(D_I1-Pad2): track 63.5 -> 73.2 mm
- net Net-(D_9-Pad2): track 42.2 -> 51.7 mm
- net Net-(D_@1-Pad2): track 69.9 -> 79.2 mm
- net Net-(D_RAlt1-Pad2): track 109.5 -> 118.5 mm
- net Net-(D_Del1-Pad2): track 57.3 -> 66.2 mm
- net Net-(D_Right1-Pad2): track 122.6 -> 131.2 mm
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Other:
- board size 313.3 x 123.8 mm -> 313.3 x 131.6 mm
