File: kicad/kbic65.sch (KiCad schematic (older format))
At the start: 150 parts, among them U1 ProMicro

Commit message: Wiring 4 life
Connections:
- net COL0: now also U1.14 (B2); no longer U1.20 (F4)
- net COL1: now also U1.13 (B6); no longer U1.19 (F5)
- net COL2: now also U1.15 (B3); no longer U1.18 (F6)
- net COL3: now also U1.16 (B1); no longer U1.17 (F7)
- net COL4: now also U1.17 (F7); no longer U1.16 (B1)
- net COL5: now also U1.18 (F6); no longer U1.15 (B3)
- net COL6: now also U1.19 (F5); no longer U1.14 (B2)
- net COL7: now also U1.20 (F4); no longer U1.13 (B6)
Changed lines of the file:
@@
 ROW0
 Text GLabel 9200 3150 1    39   Input ~ 0
+COL7
+Text GLabel 9300 3150 1    39   Input ~ 0
+COL6
+Text GLabel 9400 3150 1    39   Input ~ 0
+COL5
+Text GLabel 9500 3150 1    39   Input ~ 0
+COL4
+Text GLabel 9600 3150 1    39   Input ~ 0
+COL3
+Text GLabel 9700 3150 1    39   Input ~ 0
+COL2
+Text GLabel 9800 3150 1    39   Input ~ 0
 COL0
-Text GLabel 9300 3150 1    39   Input ~ 0
+Text GLabel 9900 3150 1    39   Input ~ 0
 COL1
-Text GLabel 9400 3150 1    39   Input ~ 0
-COL2
-Text GLabel 9500 3150 1    39   Input ~ 0
-COL3
-Text GLabel 9600 3150 1    39   Input ~ 0
-COL4
-Text GLabel 9700 3150 1    39   Input ~ 0
-COL5
-Text GLabel 9800 3150 1    39   Input ~ 0
-COL6
-Text GLabel 9900 3150 1    39   Input ~ 0
-COL7
 $Comp
 L promicro:ProMicro U1

Commit message: Completed first version of full wiring
Connections:
- net ROW0: now also U1.11 (B4); no longer U1.12 (B5)
- net ROW1: now also U1.12 (B5); no longer U1.11 (B4)
- net ROW2: now also U1.9 (D7); no longer U1.10 (E6)
- net ROW3: now also U1.10 (E6); no longer U1.9 (D7)
- net ROW4: now also U1.7 (D4); no longer U1.8 (C6)
- net ROW5: now also U1.8 (C6); no longer U1.7 (D4)
- net ROW6: now also U1.5 (SCL); no longer U1.6 (SDA)
- net ROW7: now also U1.6 (SDA); no longer U1.5 (SCL)
Changed lines of the file:
@@
 ROW8
 Text GLabel 9200 4550 3    39   Input ~ 0
+ROW6
+Text GLabel 9300 4550 3    39   Input ~ 0
 ROW7
-Text GLabel 9300 4550 3    39   Input ~ 0
-ROW6
 Text GLabel 9400 4550 3    39   Input ~ 0
+ROW4
+Text GLabel 9500 4550 3    39   Input ~ 0
 ROW5
-Text GLabel 9500 4550 3    39   Input ~ 0
-ROW4
 Text GLabel 9600 4550 3    39   Input ~ 0
+ROW2
+Text GLabel 9700 4550 3    39   Input ~ 0
 ROW3
-Text GLabel 9700 4550 3    39   Input ~ 0
-ROW2
 Text GLabel 9800 4550 3    39   Input ~ 0
+ROW0
+Text GLabel 9900 4550 3    39   Input ~ 0
 ROW1
-Text GLabel 9900 4550 3    39   Input ~ 0
-ROW0
 Text GLabel 9200 3150 1    39   Input ~ 0
 COL7

Commit message: Starting new wiring
Connections:
- net ROW0: now also U1.12 (B5); no longer U1.11 (B4)
- net ROW1: now also U1.5 (SCL); no longer U1.12 (B5)
- net ROW2: now also U1.11 (B4); no longer U1.9 (D7)
- net ROW3: now also U1.6 (SDA); no longer U1.10 (E6)
- net ROW4: now also U1.10 (E6); no longer U1.7 (D4)
- net ROW5: now also U1.7 (D4); no longer U1.8 (C6)
- net ROW6: now also U1.9 (D7); no longer U1.5 (SCL)
- net ROW7: now also U1.8 (C6); no longer U1.6 (SDA)
Changed lines of the file:
@@
 ROW8
 Text GLabel 9200 4550 3    39   Input ~ 0
+ROW1
+Text GLabel 9300 4550 3    39   Input ~ 0
+ROW3
+Text GLabel 9400 4550 3    39   Input ~ 0
+ROW5
+Text GLabel 9500 4550 3    39   Input ~ 0
+ROW7
+Text GLabel 9600 4550 3    39   Input ~ 0
 ROW6
-Text GLabel 9300 4550 3    39   Input ~ 0
-ROW7
-Text GLabel 9400 4550 3    39   Input ~ 0
+Text GLabel 9700 4550 3    39   Input ~ 0
 ROW4
-Text GLabel 9500 4550 3    39   Input ~ 0
-ROW5
-Text GLabel 9600 4550 3    39   Input ~ 0
+Text GLabel 9800 4550 3    39   Input ~ 0
 ROW2
-Text GLabel 9700 4550 3    39   Input ~ 0
-ROW3
-Text GLabel 9800 4550 3    39   Input ~ 0
+Text GLabel 9900 4550 3    39   Input ~ 0
 ROW0
-Text GLabel 9900 4550 3    39   Input ~ 0
-ROW1
 Text GLabel 9200 3150 1    39   Input ~ 0
 COL7

Commit message: Fixed 6u spacebar
Parts:
- MX_Space2_6u1: footprint MX_Only:MXOnly-6U-Centered-NoLED -> MX_Only:MXOnly-6U-NoLED
Changed lines of the file:
@@
 F 0 "MX_Space2_6u1" H 18433 11323 60  0000 C CNN
 F 1 "MX-NoLED" H 18433 11249 20  0000 C CNN
-F 2 "MX_Only:MXOnly-6U-Centered-NoLED" H 17775 11075 60  0001 C CNN
+F 2 "MX_Only:MXOnly-6U-NoLED" H 17775 11075 60  0001 C CNN
 F 3 "" H 17775 11075 60  0001 C CNN
 	1    18400 11100

Commit message: pre-updating gnd
Connections:
- net GNDREF: now reaches U1.23 (GND)
- net GNDREF: now also U1.3 (GND), U1.4 (GND)
Changed lines of the file:
@@
 Wire Wire Line
 	11500 4750 12350 4750
+$Comp
+L power:GNDREF #PWR?
+U 1 1 602F2C7C
+P 8900 5250
+F 0 "#PWR?" H 8900 5000 50  0001 C CNN
+F 1 "GNDREF" H 8905 5077 50  0000 C CNN
+F 2 "" H 8900 5250 50  0001 C CNN
+F 3 "" H 8900 5250 50  0001 C CNN
+	1    8900 5250
+	1    0    0    -1
+$EndComp
+Text GLabel 8900 5250 0    50   Input ~ 0
+GND
+Text GLabel 9000 4550 3    39   Input ~ 0
+GND
+Text GLabel 9100 4550 3    39   Input ~ 0
+GND
+Text GLabel 8900 3150 1    39   Input ~ 0
+GND
 $EndSCHEMATC

Commit message: created drawings for top window
Parts:
- D_0, D_1, D_2, D_3, D_4, D_5, D_6, D_7, D_8, D_9, D_@1, D_A1, D_B1, D_BKSLSH1, D_BkSp1, D_BkSp2, D_C1, D_Comma1, D_CpsLck1, D_D1, D_Del1, D_Dot1, D_Down1, D_E1, D_Enter1, D_Equal1, D_Esc1, D_F1, D_FwdSlsh1, D_G1, D_H1, D_Hyphen1, D_I1, D_ISO_BKSLSH1, D_J1, D_K1, D_L1, D_LAlt1, D_LBKT1, D_LCtrl1, D_LShift1, D_LWin1, D_Left1, D_M1, D_N1, D_O1, D_P1, D_PgDn1, D_PgUp1, D_Q1, D_R1, D_RAlt1, D_RBKT1, D_RCtrl1, D_RShift1, D_RWin1, D_Right1, D_S1, D_SemiCol1, D_Space1, D_T1, D_Tab1, D_Tilde1, D_U1, D_Up1, D_V1, D_W1, D_X1, D_Y1, D_Z1: symbol Device:D_Small -> kbic65-rescue:D_Small-Device
